Commit message: fix: robot dae model unable to load

File: legged_examples/legged_unitree/legged_unitree_description/urdf/robot.xacro (robot description, xacro)
@@ -8,5 +8,5 @@
     <xacro:include filename="$(find legged_unitree_description)/urdf/$(arg robot_type)/const.xacro"/>
 <!--    <xacro:property name="mesh_path" value="../meshes"/>-->
-    <xacro:property name="mesh_path" value="$(find legged_unitree_description)/meshes/$(arg robot_type)"/>
+    <xacro:property name="mesh_path" value="file://$(find legged_unitree_description)/meshes/$(arg robot_type)"/>
     <link name="base">
         <visual>
